File: 12v-2x6.kicad_sch (KiCad schematic)
At the start: 8 parts

Commit message: Update & Review
Other:
- note added: "5V / GND ------>"
- note added: "5VP / GND1 <------"
- note removed: "5V / GND"
- note removed: "5VP / GND1"
- company: eggsampler -> github.com/eggsampler
Changed lines of the file:
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@@
 	(title_block
 		(title "12V-2x6 Current Monitor")
-		(date "2025-08-12")
+		(date "2025-09-21")
 		(rev "1")
-		(company "eggsampler")
+		(company "github.com/eggsampler")
 	)
 	(text "Fan Mounts"
@@
 		)
 	)
-	(text "5VP / GND1"
+	(text "5VP / GND1\n<------"
 		(exclude_from_sim no)
-		(at 138.43 27.94 0)
+		(at 139.7 25.4 0)
 		(effects
 			(font
 				(size 1.27 1.27)
 			)
+			(justify right)
 		)
 	)
-	(text "5V / GND"
+	(text "5V / GND\n------>"
 		(exclude_from_sim no)
-		(at 153.67 27.94 0)
+		(at 152.4 25.4 0)
 		(effects
 			(font
 				(size 1.27 1.27)
 			)
+			(justify left)
 		)
 	)
