File: SHT_Connector_USB.kicad_sch (KiCad schematic)
At the start: 5 parts, among them J3 USB_C_Receptacle_USB2.0_16P, U8 USBLC6-2SC6

Commit message: Update & Review
Other:
- company: eggsampler -> github.com/eggsampler
Changed lines of the file:
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@@
 	(title_block
 		(title "12V-2x6 Current Monitor")
-		(date "2025-08-12")
+		(date "2025-09-21")
 		(rev "1")
-		(company "eggsampler")
+		(company "github.com/eggsampler")
 	)
 	(text "Ferrite Bead should be lower resistance"
