File: SHT_CurrentSense.kicad_sch (KiCad schematic)
At the start: 6 parts

Commit message: Update & Review
Other:
- company: eggsampler -> github.com/eggsampler
Changed lines of the file:
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@@
 	(title_block
 		(title "12V-2x6 Current Monitor")
-		(date "2025-08-12")
+		(date "2025-09-21")
 		(rev "1")
-		(company "eggsampler")
+		(company "github.com/eggsampler")
 	)
 	(text "\"Worst\" unbalanced case: 13V 13A per pin in 3mR\nVdrop = 13*0.003 = 0.039\nPdiss = (13^2)*0.003 = 0.507\n39mV @ 507mW\n(39mV uses almost full accuracy of INA238 +/-40.96 mV @ ADCRANGE = 1)\n\nAssuming Rtheta 40C/W\nTdelta = 0.507*40 = 20.28 above ambient\n\nWSKW0612 rated 1W @ 70*C\n1oz or 2oz CU on PCB should help dissipate\n\n10164279-124121LF max contact resistance 10mR per power pin\nLooking at 10+10+3=23mR resistance per line\nPdiss = (13^2)*0.023 = 3.887\nAlmost 3.9w worst case per line\n\nAt 8.5A operating current (approx 600W/12V/6pairs)\nPdiss = (8.5^2)*0.023 = 1.66175\n1.66W per line under operating"
