File: SHT_IO.kicad_sch (KiCad schematic)
At the start: 43 parts, among them J4 PH 1x02 2.54, J5 PH 1x02 2.54, J6 S2B-PH-K 1x02 P2, J7 S2B-PH-K 1x02 P2, J8 Conn_01x04, M2 470531000, Q1 AO3400A, SW1 SKRK, SW2 PCM12, U14 PCA9306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

Commit message: Update & Review
Parts:
- J8: now not fitted; now left out of the parts list
Other:
- note added: "10k NTC thermistors via voltage divider to 10k resistors Thermistor type to be software configurable"
- note added: "Fan circuit to drive fan from 5V usb supply Driven from MCU PWM output Provides tacho input back to MCU"
- note added: "Hardware version "number" Read by ADC For any future HW revisions SW needs to know about"
- note added: "Isolated case switch headers Designed to daisy chain to motherboard header"
- note added: "Passive buzzer Designed to be driven from IO pins PWM frequencies"
- note added: "STM32 boot mode selection switch"
- note added: "STM32 hardware reset"
- note added: "Solder jumper to allow disabling the power leds"
- note added: "Status LEDs to give outputs from MCU"
- note added: "UART programming header, not populated by default"
- company: eggsampler -> github.com/eggsampler
- moved on the sheet: C36, C37, C38, M2, R42, R43, R44, R45, R46, U14
