File: SHT_Isolation_Alert.kicad_sch (KiCad schematic)
At the start: 3 parts, among them U12 ADuM260N

Commit message: Update & Review
Parts:
- U12: value ADuM260N -> ADuM260N1
Other:
- company: eggsampler -> github.com/eggsampler
Changed lines of the file:
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@@
 	(title_block
 		(title "12V-2x6 Current Monitor")
-		(date "2025-08-12")
+		(date "2025-09-21")
 		(rev "1")
-		(company "eggsampler")
+		(company "github.com/eggsampler")
 	)
 	(text "INA238 ALERT pin is an open-drain and active-low by default, using fail safe high state as default\n\nUse ADuM260N1 so default idle state is high to match INA238"
@@
 			)
 		)
-		(property "Value" "ADuM260N"
+		(property "Value" "ADuM260N1"
 			(at 152.4 83.82 0)
 			(effects
