File: SHT_Isolation_I2C.kicad_sch (KiCad schematic)
At the start: 7 parts, among them U11 ISO1540

Commit message: Update & Review
Other:
- company: eggsampler -> github.com/eggsampler
Changed lines of the file:
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@@
 	(title_block
 		(title "12V-2x6 Current Monitor")
-		(date "2025-08-12")
+		(date "2025-09-21")
 		(rev "1")
-		(company "eggsampler")
+		(company "github.com/eggsampler")
 	)
 	(text "SDA and SCL are interchangeable as the internal circuitry for each is identical\nThese connections are swapped for PCB placement reasons\n\nISO1640 is a drop-in replacement"
