File: SHT_Isolation_Power.kicad_sch (KiCad schematic)
At the start: 5 parts, among them U10 B0505ST8-W3

Commit message: Update & Review
Other:
- company: eggsampler -> github.com/eggsampler
Changed lines of the file:
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@@
 	(title_block
 		(title "12V-2x6 Current Monitor")
-		(date "2025-08-12")
+		(date "2025-09-21")
 		(rev "1")
-		(company "eggsampler")
+		(company "github.com/eggsampler")
 	)
 	(text "Translated from datasheet\n\n电源关断管脚，接GND1芯片正常工作，接逻辑高电平，芯片停止工作。\nThe power shutdown pin - connect it to GND1 for normal operation; connect it to a logic high level to stop the chip from operating.\n\n输出电压选择。将VSEL连接到VISO以获得5 V输出或将VSEL连接到GNDISO以获得3.3 V输出。这个引脚有一个较弱的内部上拉；因此，不要让该引脚悬空。\nOutput voltage selection - connect VSEL to VISO for a 5 V output, or connect VSEL to GNDISO for a 3.3 V output. This pin has a weak internal pull-up, so it should not be left floating."
