File: SHT_MCU.kicad_sch (KiCad schematic)
At the start: 17 parts, among them U7 STM32F103C8Tx, Y1 8M YSX530GA 20pF, Y2 32.768k FC-135 12.5pF

Commit message: Update & Review
Other:
- company: eggsampler -> github.com/eggsampler
Changed lines of the file:
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@@
 	(title_block
 		(title "12V-2x6 Current Monitor")
-		(date "2025-08-12")
+		(date "2025-09-21")
 		(rev "1")
-		(company "eggsampler")
+		(company "github.com/eggsampler")
 	)
 	(text "Ferrite Bead should be higher resistance"
