File: SHT_MCU_Power.kicad_sch (KiCad schematic)
At the start: 4 parts, among them U13 MIC5219-3.3YM5

Commit message: Update & Review
Other:
- company: eggsampler -> github.com/eggsampler
Changed lines of the file:
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@@
 	(title_block
 		(title "12V-2x6 Current Monitor")
-		(date "2025-08-12")
+		(date "2025-09-21")
 		(rev "1")
-		(company "eggsampler")
+		(company "github.com/eggsampler")
 	)
 	(text "Using linear regulator not switching for less noise\nMIC5219 typically 10mV-500mV dropout, heaps of headroom from 5->3.3\n500mA should be more than enough for the STM32"
