File: SHT_TempSense.kicad_sch (KiCad schematic)
At the start: 6 parts, among them U15 TMP102xxDRL, U16 TMP102xxDRL, U17 TMP102xxDRL

Commit message: Update & Review
Other:
- company: eggsampler -> github.com/eggsampler
Changed lines of the file:
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@@
 	(title_block
 		(title "12V-2x6 Current Monitor")
-		(date "2025-08-12")
+		(date "2025-09-21")
 		(rev "1")
-		(company "eggsampler")
+		(company "github.com/eggsampler")
 	)
 	(text "Placed near the 12v-2x6 connectors to infer close temperature"
