File: 12v-2x6.kicad_pcb (KiCad board)
At the start: 6 copper layers, 100 x 67.8 mm, 152 parts, among them J1 10164279-124121LF, J2 10164279-124121LF, J3 USB_C_Receptacle_USB2.0_16P, J4 PH 1x02 2.54, J5 PH 1x02 2.54, J6 S2B-PH-K 1x02 P2, J7 S2B-PH-K 1x02 P2, J8 Conn_01x04, M2 470531000, Q1 AO3400A, SW1 SKRK, SW2 PCM12, U1 INA238, U10 B0505ST8-W3, U11 ISO1540, U12 ADuM260N, U13 MIC5219-3.3YM5, U14 PCA9306, U15 TMP102xxDRL, U16 TMP102xxDRL, U17 TMP102xxDRL, U2 INA238, U3 INA238, U4 INA238, U5 INA238, U6 INA238, U7 STM32F103C8Tx, U8 USBLC6-2SC6, U9 TLP175A, Y1 8M YSX530GA 20pF, Y2 32.768k FC-135 12.5pF

Commit message: Update & Review
Parts:
- J1, J2: footprint 12v-2x6:10164279-001LF -> 12v-2x6:10164279-124121LF
- U12: value ADuM260N -> ADuM260N1
Other:
- board text added: "2oz copper on 1.6mm Default track width 10mil/0.254mm Default spacing 0.2mm Vias 0.6mm/0.3mm & to be filled and capped GND via stitching around 12V areas is for heat transfer GND via stitching in 12V areas is for current+heat transfer"
- board text added: "JLCJLCJLCJLC"
- board text removed: "1oz or 2oz copper on 1.6mm Default track width 10mil/0.254mm Default spacing 0.2mm Vias 0.6mm/0.3mm & to be filled and capped GND via stitching around 12V areas is for heat transfer GND via stitching in 12V areas is for current+heat transfer"
Changed lines of the file:
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@@
 	(title_block
 		(title "12V-2x6 Current Monitor")
-		(date "2025-08-12")
+		(date "2025-09-21")
 		(rev "1")
+		(company "github.com/eggsampler")
 	)
 	(layers
@@
 		(sheetname "/Input Output/")
 		(sheetfile "SHT_IO.kicad_sch")
-		(attr through_hole)
+		(attr through_hole exclude_from_bom dnp)
 		(fp_line
 			(start -1.38 -1.38)
@@
 		)
 	)
-	(footprint "12v-2x6:10164279-001LF"
+	(footprint "12v-2x6:10164279-124121LF"
 		(layer "F.Cu")
 		(at 55.15 58.5 -90)
@@
 		(property "Reference" "J2"
 			(at -7 4.5 270)
-			(unlocked yes)
 			(layer "F.SilkS")
-			(hide yes)
 			(effects
 				(font
-					(size 0.8 0.8)
-					(thickness 0.1)
+					(size 1 1)
+					(thickness 0.15)
 				)
 			)
@@
 			)
 		)
-		(property "LCSC" ""
-			(at 0 0 0)
-			(layer "F.SilkS")
-			(hide yes)
-			(effects
-				(font
-					(size 1.27 1.27)
-					(thickness 0.15)
-				)
-			)
-		)
 		(sheetname "/12V-2x6 Connectors/")
 		(sheetfile "SHT_Connector_12V.kicad_sch")
@@
 			)
 		)
-		(property "Value" "ADuM260N"
+		(property "Value" "ADuM260N1"
 			(at 0 7.35 0)
 			(layer "F.Fab")
@@
 		(embedded_fonts no)
 	)
-	(footprint "12v-2x6:10164279-001LF"
+	(footprint "12v-2x6:10164279-124121LF"
 		(layer "F.Cu")
 		(at 55.15 92.5 -90)
@@
 		(tags "PCIe 12VHPWR 2x6 CEM5 Amphenol 10164279")
 		(property "Reference" "J1"
-			(at -7 4.5 90)
-			(unlocked yes)
+			(at -7 4.5 270)
 			(layer "F.SilkS")
-			(hide yes)
 			(effects
 				(font
-					(size 0.8 0.8)
-					(thickness 0.1)
+					(size 1 1)
+					(thickness 0.15)
 				)
 			)
 		)
 		(property "Value" "10164279-124121LF"
-			(at -7.5 10 90)
+			(at -7.5 10 270)
 			(layer "F.Fab")
 			(effects
@@
 		)
 		(property "Datasheet" ""
-			(at 0 0 90)
+			(at 0 0 270)
 			(layer "F.Fab")
 			(hide yes)
@@
 		)
 		(property "Description" ""
-			(at 0 0 90)
+			(at 0 0 270)
 			(layer "F.Fab")
 			(hide yes)
@@
 			)
 		)
-		(property "LCSC" ""
-			(at 0 0 0)
-			(layer "F.SilkS")
-			(hide yes)
-			(effects
-				(font
-					(size 1.27 1.27)
-					(thickness 0.15)
-				)
-			)
-		)
 		(sheetname "/12V-2x6 Connectors/")
 		(sheetfile "SHT_Connector_12V.kicad_sch")
@@
 		)
 	)
+	(gr_text "JLCJLCJLCJLC"
+		(at 85.5 46.1 0)
+		(layer "F.SilkS")
+		(effects
+			(font
+				(size 1 1)
+				(thickness 0.15)
+			)
+			(justify left bottom)
+		)
+	)
 	(gr_text "2"
 		(at 126.2 100.3 0)
@@
 		)
 	)
-	(gr_text "1oz or 2oz copper on 1.6mm\nDefault track width 10mil/0.254mm\nDefault spacing 0.2mm\nVias 0.6mm/0.3mm & to be filled and capped\n\nGND via stitching around 12V areas is for heat transfer\nGND via stitching in 12V areas is for current+heat transfer"
+	(gr_text "2oz copper on 1.6mm\nDefault track width 10mil/0.254mm\nDefault spacing 0.2mm\nVias 0.6mm/0.3mm & to be filled and capped\n\nGND via stitching around 12V areas is for heat transfer\nGND via stitching in 12V areas is for current+heat transfer"
 		(at 110 120 0)
 		(layer "User.1")
@@
 	)
 	(segment
-		(start 52.8125 97.5)
-		(end 53.5 97.5)
-		(width 0.254)
-		(layer "F.Cu")
-		(net 104)
-	)
-	(segment
 		(start 50.6 38.5)
 		(end 48.7 40.4)
@@
 	)
 	(segment
-		(start 53.5 97.5)
-		(end 54 97)
-		(width 0.254)
-		(layer "F.Cu")
-		(net 104)
-	)
-	(segment
 		(start 91 57.4)
 		(end 91 56.8)
@@
 	)
 	(segment
+		(start 59.488127 94.4)
+		(end 64.4 94.4)
+		(width 0.254)
+		(layer "F.Cu")
+		(net 104)
+	)
+	(segment
+		(start 101 74.7)
+		(end 101 73.6)
+		(width 0.254)
+		(layer "F.Cu")
+		(net 104)
+	)
+	(segment
 		(start 49.6 96.7)
 		(end 48.7 95.8)
@@
 	)
 	(segment
+		(start 92.45 99)
+		(end 105 86.45)
+		(width 0.254)
+		(layer "F.Cu")
+		(net 104)
+	)
+	(segment
 		(start 48.7 95.8)
 		(end 48.7 68.5)
@@
 	)
 	(segment
+		(start 64.4 94.4)
+		(end 69 99)
+		(width 0.254)
+		(layer "F.Cu")
+		(net 104)
+	)
+	(segment
 		(start 96.8 76.5)
 		(end 96.8 74.3)
@@
 	)
 	(segment
-		(start 105 78.7)
-		(end 101 74.7)
+		(start 56.388127 97.5)
+		(end 59.488127 94.4)
 		(width 0.254)
 		(layer "F.Cu")
@@
 	)
 	(segment
-		(start 56.888127 97)
-		(end 59.488127 94.4)
-		(width 0.254)
-		(layer "F.Cu")
-		(net 104)
-	)
-	(segment
 		(start 98.01 73.09)
 		(end 100.49 73.09)
@@
 	)
 	(segment
+		(start 105 78.7)
+		(end 101 74.7)
+		(width 0.254)
+		(layer "F.Cu")
+		(net 104)
+	)
+	(segment
 		(start 94.7 78.6)
 		(end 96.8 76.5)
@@
 	)
 	(segment
-		(start 101 74.7)
-		(end 101 73.6)
+		(start 91.2 56.6)
+		(end 92.2 56.6)
 		(width 0.254)
 		(layer "F.Cu")
@@
 	)
 	(segment
-		(start 91.2 56.6)
-		(end 92.2 56.6)
+		(start 92.2 57.6)
+		(end 91.2 57.6)
 		(width 0.254)
 		(layer "F.Cu")
@@
 	)
 	(segment
-		(start 92.2 57.6)
-		(end 91.2 57.6)
+		(start 69 99)
+		(end 92.45 99)
 		(width 0.254)
 		(layer "F.Cu")
@@
 	)
 	(segment
-		(start 92.45 99)
-		(end 105 86.45)
-		(width 0.254)
-		(layer "F.Cu")
-		(net 104)
-	)
-	(segment
-		(start 105 86.45)
-		(end 105 78.7)
-		(width 0.254)
-		(layer "F.Cu")
-		(net 104)
-	)
-	(segment
 		(start 92.2 70.8)
 		(end 91.2 70.8)
@@
 	)
 	(segment
-		(start 64.4 94.4)
-		(end 69 99)
-		(width 0.254)
-		(layer "F.Cu")
-		(net 104)
-	)
-	(segment
-		(start 54 97)
-		(end 56.888127 97)
-		(width 0.254)
-		(layer "F.Cu")
-		(net 104)
-	)
-	(segment
-		(start 59.488127 94.4)
-		(end 64.4 94.4)
+		(start 105 86.45)
+		(end 105 78.7)
 		(width 0.254)
 		(layer "F.Cu")
@@
 	)
 	(segment
-		(start 94.725735 65.6)
-		(end 94.725735 65.5)
+		(start 52.8125 97.5)
+		(end 56.388127 97.5)
 		(width 0.254)
 		(layer "F.Cu")
@@
 	)
 	(segment
-		(start 69 99)
-		(end 92.45 99)
+		(start 94.725735 65.6)
+		(end 94.725735 65.5)
 		(width 0.254)
 		(layer "F.Cu")

Commit message: Minor updates
Ground changes, small updates
Parts:
- removed kibuzzard-689AF453: G***, kibuzzard-689AF453
- added kibuzzard-68F03828: G***, kibuzzard-68F03828, F.Cu at (92.1, 38.7)
- moved SYM1 2.60 mm to (89.6, 94.1)
Connections:
- J1 pad 10: GND1 -> /12V-2x6 Connectors/GND_12V_4
- J1 pad 11: GND1 -> /12V-2x6 Connectors/GND_12V_5
- J1 pad 12: GND1 -> /12V-2x6 Connectors/GND_12V_6
- J1 pad 7: GND1 -> /12V-2x6 Connectors/GND_12V_1
- J1 pad 8: GND1 -> /12V-2x6 Connectors/GND_12V_2
- J1 pad 9: GND1 -> /12V-2x6 Connectors/GND_12V_3
- J2 pad 10: GND1 -> /12V-2x6 Connectors/GND_12V_3
- J2 pad 11: GND1 -> /12V-2x6 Connectors/GND_12V_2
- J2 pad 12: GND1 -> /12V-2x6 Connectors/GND_12V_1
- J2 pad 7: GND1 -> /12V-2x6 Connectors/GND_12V_6
- J2 pad 8: GND1 -> /12V-2x6 Connectors/GND_12V_5
- J2 pad 9: GND1 -> /12V-2x6 Connectors/GND_12V_4
Routing:
- net /Current Sensing/CurrentSense6/IN-: track 35.2 -> 33.3 mm
- net /12V-2x6 Connectors/12V_OUT6: track 40.3 -> 38.4 mm, vias 11 -> 7
- net /Current Sensing/CurrentSense1/IN+: track 16.7 -> 14.9 mm
- net /Current Sensing/CurrentSense6/IN+: track 34.7 -> 33.0 mm
- net /12V-2x6 Connectors/12V_OUT5: track 31.7 -> 32.9 mm, vias 11 -> 7
- net /Current Sensing/CurrentSense1/IN-: track 16.7 -> 15.7 mm
- net /Current Sensing/CurrentSense5/IN+: track 26.3 -> 27.1 mm
- net /Current Sensing/CurrentSense5/IN-: track 26.8 -> 27.6 mm
- net /12V-2x6 Connectors/12V_OUT1: track 21.4 -> 20.7 mm, vias 10 -> 6
- net /12V-2x6 Connectors/12V_OUT3: track 21.2 -> 21.6 mm, vias 11 -> 7
- net /12V-2x6 Connectors/12V_OUT4: track 24.8 -> 25.0 mm, vias 11 -> 7
- net /12V-2x6 Connectors/12V_OUT2: track 21.6 -> 21.9 mm, vias 11 -> 7
- net GND1: vias 213 -> 224
- net /12V-2x6 Connectors/GND_12V_6: vias 0 -> 10
- net /12V-2x6 Connectors/GND_12V_5: vias 0 -> 12
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- added copper zone on B.Cu, net /12V-2x6 Connectors/GND_12V_1
- added copper zone on In1.Cu, net /12V-2x6 Connectors/GND_12V_1
- added copper zone on In3.Cu, net /12V-2x6 Connectors/GND_12V_1
- added copper zone on B.Cu, net /12V-2x6 Connectors/GND_12V_2
- added copper zone on In1.Cu, net /12V-2x6 Connectors/GND_12V_2
- added copper zone on In3.Cu, net /12V-2x6 Connectors/GND_12V_2
- added copper zone on B.Cu, net /12V-2x6 Connectors/GND_12V_3
- added copper zone on In1.Cu, net /12V-2x6 Connectors/GND_12V_3
- added copper zone on In3.Cu, net /12V-2x6 Connectors/GND_12V_3
- added copper zone on B.Cu, net /12V-2x6 Connectors/GND_12V_4
- added copper zone on In1.Cu, net /12V-2x6 Connectors/GND_12V_4
- added copper zone on In3.Cu, net /12V-2x6 Connectors/GND_12V_4
- added copper zone on B.Cu, net /12V-2x6 Connectors/GND_12V_5
- added copper zone on In1.Cu, net /12V-2x6 Connectors/GND_12V_5
- added copper zone on In3.Cu, net /12V-2x6 Connectors/GND_12V_5
- added copper zone on B.Cu, net /12V-2x6 Connectors/GND_12V_6
- added copper zone on In1.Cu, net /12V-2x6 Connectors/GND_12V_6
- added copper zone on In3.Cu, net /12V-2x6 Connectors/GND_12V_6
Other:
- board text removed: "JLCJLCJLCJLC"
