File: SHT_Connector_12V.kicad_sch (KiCad schematic)
At the start: 2 parts, among them J1 10164279-124121LF, J2 10164279-124121LF

Commit message: Update & Review
Parts:
- J1, J2: footprint 12v-2x6:10164279-001LF -> 12v-2x6:10164279-124121LF
Other:
- company: eggsampler -> github.com/eggsampler
Changed lines of the file:
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@@
 	(title_block
 		(title "12V-2x6 Current Monitor")
-		(date "2025-08-12")
+		(date "2025-09-21")
 		(rev "1")
-		(company "eggsampler")
+		(company "github.com/eggsampler")
 	)
 	(text "These are reversed\nto the inputs\non purpose"
@@
 			)
 		)
-		(property "Footprint" "12v-2x6:10164279-001LF"
+		(property "Footprint" "12v-2x6:10164279-124121LF"
 			(at 59.69 36.83 0)
 			(effects
@@
 			)
 		)
-		(property "Footprint" "12v-2x6:10164279-001LF"
+		(property "Footprint" "12v-2x6:10164279-124121LF"
 			(at 59.69 125.73 0)
 			(effects

Commit message: Minor updates
Ground changes, small updates
Connections:
- removed net GND1: J1.10 (GND), J1.11 (GND), J1.12 (GND), J1.7 (GND), J1.8 (GND), J1.9 (GND), J2.10 (GND), J2.11 (GND), J2.12 (GND), J2.7 (GND), J2.8 (GND), J2.9 (GND)
- new net GND_12V_1: J1.7 (GND), J2.12 (GND)
- new net GND_12V_2: J1.8 (GND), J2.11 (GND)
- new net GND_12V_3: J1.9 (GND), J2.10 (GND)
- new net GND_12V_4: J1.10 (GND), J2.9 (GND)
- new net GND_12V_5: J1.11 (GND), J2.8 (GND)
- new net GND_12V_6: J1.12 (GND), J2.7 (GND)
